File: files/ch340g/fabftdi-ch340g.sch (EAGLE design)
At the start: 12 parts, among them U1 CH340G, Y1 12MHz

Commit message: updated all files, added components list
Other:
- moved on the sheet: C1, C2, D1, D2, JP1, R1
