File: files/mega8/fabftdi-mega8.brd (EAGLE design)
At the start: 64.8 x 31.4 mm, 15 parts, among them J1 ISP, J2 FTDI-SMD-HEADER, Q1 12MHz, U1 ATmega8A-AU, U2 USB_MINI

Commit message: updated all files, added components list
Parts:
- R2, R3: value 68 -> 49
- moved J2 4.45 mm to (54.6, 16.5)
- moved J1 3.81 mm to (45.8, 16.9)
- moved C2 1.91 mm to (41.8, 7.62)
- moved C3 1.91 mm to (18.9, 22.9)
- moved Q1 1.91 mm to (30.7, 7.62)
- moved R6 1.91 mm to (46.9, 7.62)
- moved U1 1.91 mm to (32.4, 19.0)
- moved D1 1.90 mm to (13.3, 22.9)
- moved C1 1.90 mm to (19.1, 7.62)
- moved R1 1.90 mm to (16.1, 22.9)
- moved R2 1.90 mm to (19.1, 13.3)
- moved R3 1.90 mm to (19.1, 17.4)
- moved R4 1.90 mm to (22.2, 22.9)
- moved R5 1.90 mm to (24.6, 22.9)
Routing:
- net N$11: track 56.9 -> 109.2 mm
- net N$15: track 191.8 -> 177.0 mm
- net N$13: track 92.4 -> 87.3 mm
- net GND: track 124.8 -> 120.3 mm
- net VCC: track 87.5 -> 84.9 mm
- net N$14: track 58.3 -> 56.3 mm
- net N$9: track 20.8 -> 18.9 mm
- net N$7: track 23.1 -> 21.2 mm
- net N$10: track 21.1 -> 19.1 mm
- net N$6: track 9.49 -> 7.58 mm
- net N$8: track 11.3 -> 9.44 mm
- net N$5: track 9.84 -> 7.93 mm
- net N$12: track 7.68 -> 9.59 mm
- net N$2: track 21.8 -> 21.1 mm
Other:
- board size 64.8 x 31.4 mm -> 59 x 29.5 mm
- board text added: "Fab FTDI"
- board text removed: "FABFTDI"
